Commit message: Your commit message here

File: gp_description/urdf/ballbot1.urdf.xacro (robot description, xacro)
@@ -50,8 +50,7 @@
     </visual>
     <collision>
-      <origin xyz="0 0 0" rpy="0 0 0" />
-      <geometry>
-        <mesh
-          filename="package://gp_description/meshes/base_link.STL" />
+      <origin xyz="0 0 0.35" rpy="0 0 0"/>
+      <geometry>
+        <box size="0.40 0.40 0.70"/>
       </geometry>
     </collision>
@@ -77,5 +76,5 @@
       <origin xyz="0 0 0" rpy="0 0 0" />
       <geometry>
-        <sphere radius="0.15" />
+        <sphere radius="0.125" />
       </geometry>
     </collision>
@@ -95,18 +94,15 @@
     </inertial>
   </link>
-  <joint name="sphere_roll" type="continuous">
-    <parent link="base_link" />
-    <child link="dummy_rx" />
-    <axis xyz="1 0 0" />
-  </joint>
-  <joint name="sphere_pitch" type="continuous">
-    <parent link="dummy_rx" />
-    <child link="dummy_ry" />
-    <axis xyz="0 1 0" />
-  </joint>
-  <joint name="sphere_yaw" type="continuous">
-    <parent link="dummy_ry" />
-    <child link="Sphere" />
-    <axis xyz="0 0 1" />
+  <joint name="sphere_roll" type="fixed">
+    <parent link="base_link"/>
+    <child link="dummy_rx"/>
+  </joint>
+  <joint name="sphere_pitch" type="fixed">
+    <parent link="dummy_rx"/>
+    <child link="dummy_ry"/>
+  </joint>
+  <joint name="sphere_yaw" type="fixed">
+    <parent link="dummy_ry"/>
+    <child link="Sphere"/>
   </joint>
   <link name="wheel1">
